Commit message: working basis of robot

File: src/basic_mobile_robot/models/omni_featter.urdf (robot description, URDF)
Before this commit: robot OMNIFEATTER, 5 links, 4 joints
Links:
- removed link L_B_WHEEL
- removed link L_F_WHEEL
- removed link R_B_WHEEL
- removed link R_F_WHEEL
- link BASE_LINK: geometry collision box size=${BASE_LENGHT} ${BASE_WIDTH} ${BASE_HEIGHT}; visual box size=${BASE_LENGHT} ${BASE_WIDTH} ${BASE_HEIGHT}
Joints:
- joint BASE_LINK_TO_L_B_WHEEL: axis 0 1 0 -> 0 0 1; origin xyz=-${BASE_LENGHT/2} -${BASE_WIDTH/2} -${BASE_HEIGHT/2} -> xyz=-${BASE_LENGHT/2} ${BASE_WIDTH/2+MECANUM_WHEEL_WIDTH/2} -${BASE_HEIGHT/2}  rpy=${-pi/2} 0 0
- joint BASE_LINK_TO_L_F_WHEEL: axis 0 1 0 -> 0 0 1; origin xyz=${BASE_LENGHT/2} ${BASE_WIDTH/2} ${BASE_HEIGHT/2} -> xyz=${BASE_LENGHT/2} ${BASE_WIDTH/2+MECANUM_WHEEL_WIDTH/2} -${BASE_HEIGHT/2} rpy=${-pi/2} 0 0
- joint BASE_LINK_TO_R_B_WHEEL: axis 0 1 0 -> 0 0 1; origin xyz=-${BASE_LENGHT/2} -${BASE_WIDTH/2} -${BASE_HEIGHT/2} -> xyz=-${BASE_LENGHT/2} -${BASE_WIDTH/2+MECANUM_WHEEL_WIDTH/2} -${BASE_HEIGHT/2} rpy=${pi/2} 0 0
- joint BASE_LINK_TO_R_F_WHEEL: axis 0 1 0 -> 0 0 1; origin xyz=${BASE_LENGHT/2} ${BASE_WIDTH/2} ${BASE_HEIGHT/2} -> xyz=${BASE_LENGHT/2} -${BASE_WIDTH/2+MECANUM_WHEEL_WIDTH/2} -${BASE_HEIGHT/2} rpy=${pi/2} 0 0

Commit message: temporary

File: src/basic_mobile_robot/models/omni_featter.urdf (robot description, URDF)
Before this commit: robot OMNIFEATTER, 1 links, 4 joints
Joints:
- removed joint BASE_LINK_TO_L_B_WHEEL
- removed joint BASE_LINK_TO_L_F_WHEEL
- removed joint BASE_LINK_TO_R_B_WHEEL
- removed joint BASE_LINK_TO_R_F_WHEEL
- added joint base_to_L_B_WHEEL_joint: type revolute, parent BASE_LINK, child L_B_WHEEL, origin xyz=${BASE_LENGHT/2} ${BASE_WIDTH/2+MECANUM_WHEEL_WIDTH/2} -${BASE_HEIGHT/2} rpy=${-pi/2} 0 0, axis 0 0 1, limit effort=${MECANUM_WHEEL_MAX_EFFORT} velocity=${MECANUM_WHEEL_MAX_JOINT_VEL}
- added joint base_to_L_F_WHEEL_joint: type revolute, parent BASE_LINK, child L_F_WHEEL, origin xyz=${BASE_LENGHT/2} ${BASE_WIDTH/2+MECANUM_WHEEL_WIDTH/2} -${BASE_HEIGHT/2} rpy=${-pi/2} 0 0, axis 0 0 1, limit effort=${MECANUM_WHEEL_MAX_EFFORT} velocity=${MECANUM_WHEEL_MAX_JOINT_VEL}
- added joint base_to_R_B_WHEEL_joint: type revolute, parent BASE_LINK, child R_B_WHEEL, origin xyz=${BASE_LENGHT/2} ${BASE_WIDTH/2+MECANUM_WHEEL_WIDTH/2} -${BASE_HEIGHT/2} rpy=${pi/2} 0 0, axis 0 0 1, limit effort=${MECANUM_WHEEL_MAX_EFFORT} velocity=${MECANUM_WHEEL_MAX_JOINT_VEL}
- added joint base_to_R_F_WHEEL_joint: type revolute, parent BASE_LINK, child R_F_WHEEL, origin xyz=${BASE_LENGHT/2} ${BASE_WIDTH/2+MECANUM_WHEEL_WIDTH/2} -${BASE_HEIGHT/2} rpy=${pi/2} 0 0, axis 0 0 1, limit effort=${MECANUM_WHEEL_MAX_EFFORT} velocity=${MECANUM_WHEEL_MAX_JOINT_VEL}

Commit message: Fixed error in wheels loading

File: src/basic_mobile_robot/models/omni_featter.urdf (robot description, URDF)
Before this commit: robot OMNIFEATTER, 1 links, 4 joints
Joints:
- removed joint base_to_L_B_WHEEL_joint
- removed joint base_to_L_F_WHEEL_joint
- removed joint base_to_R_B_WHEEL_joint
- removed joint base_to_R_F_WHEEL_joint

Commit message: inertia tensors applied to model for use in gazebo

File: src/basic_mobile_robot/models/omni_featter.urdf (robot description, URDF)
Before this commit: robot OMNIFEATTER, 1 links, 0 joints
Links:
- removed link BASE_LINK
