Commit message: imu gazebo simulation (not finnished)

File: src/omni_featter/omni_featter_description/urdf/base.urdf.xacro (robot description, xacro)
@@ -23,6 +23,6 @@
       <inertial>
         <origin xyz="0 0 0" rpy="0 0 0" />
-        <mass value="${MECANUM_WHEEL_MASS}" />
-        <inertia ixx="${ROBOT_MASS-MECANUM_WHEEL_MASS*(BASE_WIDTH*BASE_WIDTH+BASE_HEIGHT*BASE_HEIGHT)/12}" ixy="0" ixz="0" iyy="${ROBOT_MASS-MECANUM_WHEEL_MASS*(BASE_LENGHT*BASE_LENGHT+BASE_HEIGHT*BASE_HEIGHT)/12}" iyz="0" izz="${ROBOT_MASS-MECANUM_WHEEL_MASS*(BASE_LENGHT*BASE_LENGHT+BASE_HEIGHT*BASE_HEIGHT)/12}" />
+        <mass value="${ROBOT_MASS-MECANUM_WHEEL_MASS}" />
+        <xacro:box_inertia m="${ROBOT_MASS-MECANUM_WHEEL_MASS}" x="${BASE_LENGHT}" y="${BASE_WIDTH}" z="${BASE_HEIGHT}" />
       </inertial>
     </link>

File: src/omni_featter/omni_featter_description/urdf/omni_featter.urdf.xacro (robot description, xacro)
@@ -33,6 +33,6 @@
   <!-- ******************** MECANUM WHEELS ********************  -->
   <xacro:include filename="$(find omni_featter_description)/urdf/wheels_urdf/mecanum_wheels_macro.urdf.xacro" />
-  <!-- ******************* INERTIAL MACROS  *******************  -->
-  <xacro:include filename="$(find omni_featter_description)/urdf/basic_macros/inertial_macros.urdf.xacro" />
+  <!-- ******************* IMU LINK *******************  -->
+  <xacro:include filename="$(find omni_featter_description)/urdf/sensors/imu_.urdf.xacro" />
   <!-- ********************************************************  -->
   <!-- ****************** ASSEMBLY ****************************  -->
@@ -103,3 +103,5 @@
   BASE_LINK="BASE_LINK"
   WHEEL_MASS="${MECANUM_WHEEL_MASS}"/>
+  <!-- ****************** IMU LINK *******************************  -->
+  <xacro:Imu_link/>
 </robot>

File: src/omni_featter/omni_featter_description/urdf/wheels_urdf/mecanum_wheels_macro.urdf.xacro (robot description, xacro)
@@ -26,5 +26,5 @@
         <origin xyz="0 0 0" rpy="0 0 0" />
         <mass value="${WHEEL_MASS}" />
-        <inertia ixx="${WHEEL_MASS*(3*DIAMETER/2*DIAMETER/2+MECANUM_WHEEL_WIDTH*MECANUM_WHEEL_WIDTH)/12}" ixy="0" ixz="0" iyy="${WHEEL_MASS*(3*DIAMETER/2*DIAMETER/2+MECANUM_WHEEL_WIDTH*MECANUM_WHEEL_WIDTH)/12}" iyz="0" izz="${WHEEL_MASS*DIAMETER/2*DIAMETER/2/2}" />
+        <xacro:cylinder_inertia m="${MECANUM_WHEEL_MASS}" h="${MECANUM_WHEEL_WIDTH}" r="${DIAMETER/2}"/>
       </inertial>
     </link>
