Commit message: tri_sensor setup done: middle left and right topic

File: src/swarm_process_robot/process_robot_description/urdf/process_robot.urdf.xacro (robot description, xacro)
@@ -3,5 +3,7 @@
   <!-- Custom made macros -->
   <xacro:include filename="$(find process_robot_description)/urdf/process_robot_properties.urdf.xacro" />
-  <xacro:include filename="$(find process_robot_description)/urdf/sensors/tri_ir_sensor.urdf.xacro" />
+  <xacro:include filename="$(find process_robot_description)/urdf/sensors/tri_ir_sensor/tri_ir_sensor_middle.urdf.xacro" />
+  <xacro:include filename="$(find process_robot_description)/urdf/sensors/tri_ir_sensor/tri_ir_sensor_left.urdf.xacro" />
+  <xacro:include filename="$(find process_robot_description)/urdf/sensors/tri_ir_sensor/tri_ir_sensor_right.urdf.xacro" />
   <xacro:include filename="$(find process_robot_description)/urdf/sensors/web_cam.urdf.xacro" />
   <!-- linorobot2 macros -->
@@ -12,4 +14,5 @@
   <xacro:include filename="$(find linorobot2_description)/urdf/sensors/depth_sensor.urdf.xacro" />
   <xacro:include filename="$(find linorobot2_description)/urdf/controllers/omni_drive.urdf.xacro" />
+  <!-- Assembly of robot -->
   <xacro:base
     length="${base_length}"
@@ -19,5 +22,5 @@
     wheel_radius="${wheel_radius}"
     wheel_pos_z="${wheel_pos_z}"
-/>
+    />
   <xacro:mecanum_wheel
     side="front_left"
@@ -28,5 +31,5 @@
     pos_z="${wheel_pos_z}"
     mass="${wheel_mass}"
-  />
+    />
   <xacro:mecanum_wheel
     side="front_right"
@@ -37,5 +40,5 @@
     pos_z="${wheel_pos_z}"
     mass="${wheel_mass}"
-  />
+    />
   <xacro:mecanum_wheel
     side="rear_left"
@@ -46,5 +49,5 @@
     pos_z="${wheel_pos_z}"
     mass="${wheel_mass}"
-  />
+    />
   <xacro:mecanum_wheel
     side="rear_right"
@@ -55,7 +58,9 @@
     pos_z="${wheel_pos_z}"
     mass="${wheel_mass}"
-  />
+    />
   <xacro:imu/>
   <xacro:tri_ir_sensor x="${base_length/2}" y="0" z="${-base_height/2}" roll="0" pitch="0" yaw="0" />
+  <xacro:left_tri_ir_sensor x="${base_length/2}" y="0" z="${-base_height/2}" roll="0" pitch="0" yaw="0" />
+  <xacro:right_tri_ir_sensor x="${base_length/2}" y="0" z="${-base_height/2}" roll="0" pitch="0" yaw="0" />
   <xacro:web_cam x="${base_length/2}" y="0" z="${base_height/2}" roll="0" pitch="0" yaw="0" />
   <xacro:omni_drive_controller/>

File: src/swarm_process_robot/process_robot_description/urdf/process_robot_properties.urdf.xacro (robot description, xacro)
@@ -12,9 +12,3 @@
   <xacro:property name="wheel_mass" value=".4" />
   <xacro:property name="wheel_torque" value="20" />
-  <xacro:property name="laser_pose">
-    <origin xyz="-0.0475 0 0.125" rpy="0 0 0"/>
-  </xacro:property>
-  <xacro:property name="depth_sensor_pose">
-    <origin xyz="0.2375 0 0.06" rpy="0 0 0"/>
-  </xacro:property>
 </robot>

File: src/swarm_process_robot/process_robot_description/urdf/sensors/tri_ir_sensor/tri_ir_sensor_left.urdf.xacro (robot description, xacro)
@@ -1,5 +1,5 @@
 <robot xmlns:xacro="http://ros.org/wiki/xacro">
-    <xacro:macro name="tri_ir_sensor" params="x y z roll pitch yaw">
-        <link name="tri_ir_sensor">
+    <xacro:macro name="left_tri_ir_sensor" params="x y z roll pitch yaw">
+        <link name="left_tri_ir_sensor">
             <collision>
                 <origin xyz="0 0 0" rpy="0 0 0" />
@@ -20,19 +20,19 @@
             </inertial>
         </link>
-        <joint name="tri_ir_sensor_joint" type="fixed">
+        <joint name="left_tri_ir_sensor_joint" type="fixed">
             <axis xyz="0 0 0" />
             <origin rpy="${roll} ${pitch} ${yaw}"  xyz="${x} ${y} ${z}" />
             <parent link="base_link" />
-            <child link="tri_ir_sensor" />
+            <child link="left_tri_ir_sensor" />
         </joint>
-        <link name="tri_ir_range_frame"/>
-        <joint name="tri_ir_range_joint" type="fixed">
+        <link name="left_tri_ir_range_frame"/>
+        <joint name="left_tri_ir_range_joint" type="fixed">
             <axis xyz="0 0 0" />
             <origin rpy="0 0 0" xyz="${0.01/2} 0 0" />
-            <parent link="tri_ir_sensor" />
-            <child link="tri_ir_range_frame" />
+            <parent link="left_tri_ir_sensor" />
+            <child link="left_tri_ir_range_frame" />
         </joint>
-        <gazebo reference="tri_ir_sensor">
-            <sensor name="ir_sensor" type="ray">
+        <gazebo reference="left_tri_ir_sensor">
+            <sensor name="left_ir_sensor" type="ray">
                 <always_on>true</always_on>
                 <visualize>true</visualize>
@@ -43,5 +43,5 @@
                             <samples>360</samples>
                             <resolution>1.000000</resolution>
-                            <min_angle>-1.3962634</min_angle>
+                            <min_angle>0.523598776</min_angle>
                             <max_angle>1.3962634</max_angle>
                         </horizontal>
@@ -61,8 +61,8 @@
                 <plugin name="gazebo_ros_range" filename="libgazebo_ros_ray_sensor.so">
                     <ros>
-                        <remapping>~/out:=range</remapping>
+                        <remapping>~/out:=tri_ir_sensor/left/range</remapping>
                     </ros>
                     <output_type>sensor_msgs/Range</output_type>
-                    <frame_name>tri_ir_range_frame</frame_name>
+                    <frame_name>left_tri_ir_range_frame</frame_name>
                     <radiation>INFRARED</radiation>
                 </plugin>

Commit message: sensors are fixed

File: src/swarm_process_robot/process_robot_description/urdf/process_robot.urdf.xacro (robot description, xacro)
@@ -9,4 +9,5 @@
   <xacro:include filename="$(find process_robot_description)/urdf/controllers/omni_drive.urdf.xacro" />
   <xacro:include filename="$(find process_robot_description)/urdf/sensors/imu.urdf.xacro" />
+  <xacro:include filename="$(find process_robot_description)/urdf/sensors/lidar.urdf.xacro" />
   <!-- linorobot2 macros -->
   <xacro:include filename="$(find linorobot2_description)/urdf/mech/base.urdf.xacro" />
@@ -65,3 +66,4 @@
   <xacro:web_cam x="${base_length/2}" y="0" z="${base_height/2}" roll="0" pitch="0" yaw="0" />
   <xacro:omni_drive_controller/>
+  <xacro:lidar/>
 </robot>

File: src/swarm_process_robot/process_robot_description/urdf/sensors/imu.urdf.xacro (robot description, xacro)
@@ -20,6 +20,5 @@
           <topicName>imu/data</topicName>
           <bodyName>imu_link</bodyName>
-          <updateRateHZ>10.0</updateRateHZ>
-          <gaussianNoise>0.0</gaussianNoise>
+          <updateRateHZ>100.0</updateRateHZ>
           <xyzOffset>0 0 0</xyzOffset>
           <rpyOffset>0 0 0</rpyOffset>

File: src/swarm_process_robot/process_robot_description/urdf/sensors/tri_ir_sensor/tri_ir_sensor_left.urdf.xacro (robot description, xacro)
@@ -22,5 +22,5 @@
         <joint name="left_tri_ir_sensor_joint" type="fixed">
             <axis xyz="0 0 0" />
-            <origin rpy="${roll} ${pitch} ${yaw}"  xyz="${x} ${y} ${z}" />
+            <origin rpy="${roll} ${pitch} 0.959931089"  xyz="${x} ${y} ${z}" />
             <parent link="base_link" />
             <child link="left_tri_ir_sensor" />
@@ -44,6 +44,6 @@
                             <samples>360</samples>
                             <resolution>1.000000</resolution>
-                            <min_angle>0.523598776</min_angle>
-                            <max_angle>1.3962634</max_angle>
+                            <min_angle>-0.523598776</min_angle>
+                            <max_angle>0.523598776</max_angle>
                         </horizontal>
                     </scan>
@@ -53,9 +53,4 @@
                         <resolution>0.015000</resolution>
                     </range>
-                    <noise>
-                        <type>gaussian</type>
-                        <mean>0.0</mean>
-                        <stddev>0.01</stddev>
-                    </noise>
                     <radiation_type>INFRARED</radiation_type>
                 </ray>

File: src/swarm_process_robot/process_robot_description/urdf/sensors/tri_ir_sensor/tri_ir_sensor_middle.urdf.xacro (robot description, xacro)
@@ -53,9 +53,4 @@
                         <resolution>0.015000</resolution>
                     </range>
-                    <noise>
-                        <type>gaussian</type>
-                        <mean>0.0</mean>
-                        <stddev>0.01</stddev>
-                    </noise>
                     <radiation_type>INFRARED</radiation_type>
                 </ray>

File: src/swarm_process_robot/process_robot_description/urdf/sensors/tri_ir_sensor/tri_ir_sensor_right.urdf.xacro (robot description, xacro)
@@ -22,5 +22,5 @@
         <joint name="right_tri_ir_sensor_joint" type="fixed">
             <axis xyz="0 0 0" />
-            <origin rpy="${roll} ${pitch} ${yaw}"  xyz="${x} ${y} ${z}" />
+            <origin rpy="${roll} ${pitch} -0.959931089"  xyz="${x} ${y} ${z}" />
             <parent link="base_link" />
             <child link="right_tri_ir_sensor" />
@@ -44,5 +44,5 @@
                             <resolution>1.000000</resolution>
                             <min_angle>-0.523598776</min_angle>
-                            <max_angle>-1.3962634</max_angle>
+                            <max_angle>0.523598776</max_angle>
                         </horizontal>
                     </scan>
@@ -52,9 +52,4 @@
                         <resolution>0.015000</resolution>
                     </range>
-                    <noise>
-                        <type>gaussian</type>
-                        <mean>0.0</mean>
-                        <stddev>0.01</stddev>
-                    </noise>
                     <radiation_type>INFRARED</radiation_type>
                 </ray>

Commit message: Optimized costmap + configured controller using omni directional wheels

File: src/swarm_process_robot/process_robot_description/urdf/process_robot.urdf.xacro (robot description, xacro)
@@ -61,7 +61,7 @@
     />
   <xacro:imu/>
-  <xacro:tri_ir_sensor x="${base_length/2}" y="0" z="${-base_height/2}" roll="0" pitch="0" yaw="0" />
-  <xacro:left_tri_ir_sensor x="${base_length/2}" y="0" z="${-base_height/2}" roll="0" pitch="0" yaw="0" />
-  <xacro:right_tri_ir_sensor x="${base_length/2}" y="0" z="${-base_height/2}" roll="0" pitch="0" yaw="0" />
+  <xacro:tri_ir_sensor x="${base_length/2-0.20000}" y="0" z="${base_height/2+0.010}" roll="0" pitch="0" yaw="0" />
+  <xacro:left_tri_ir_sensor x="${base_length/2-0.20000}" y="0.01" z="${base_height/2+0.010}" roll="0" pitch="0" yaw="0" />
+  <xacro:right_tri_ir_sensor x="${base_length/2-0.20000}" y="-0.01" z="${base_height/2+0.010}" roll="0" pitch="0" yaw="0" />
   <xacro:web_cam x="${base_length/2}" y="0" z="${base_height/2}" roll="0" pitch="0" yaw="0" />
   <xacro:omni_drive_controller/>

File: src/swarm_process_robot/process_robot_description/urdf/sensors/imu.urdf.xacro (robot description, xacro)
@@ -11,5 +11,5 @@
       <sensor name="imu_sensor" type="imu">
       <always_on>true</always_on>
-      <update_rate>20</update_rate>
+      <update_rate>100</update_rate>
       <visualize>true</visualize>
       <topic>__default_topic__</topic>

File: src/swarm_process_robot/process_robot_description/urdf/sensors/tri_ir_sensor/tri_ir_sensor_left.urdf.xacro (robot description, xacro)
@@ -29,13 +29,13 @@
         <joint name="left_tri_ir_range_joint" type="fixed">
             <axis xyz="0 0 0" />
-            <origin rpy="0 0 0" xyz="${0.01/2} 0 0" />
+            <origin rpy="0 0 0" xyz="${0.01/2+0.001} 0 0" />
             <parent link="left_tri_ir_sensor" />
             <child link="left_tri_ir_range_frame" />
         </joint>
-        <gazebo reference="left_tri_ir_sensor">
+        <gazebo reference="left_tri_ir_range_frame">
             <sensor name="left_ir_sensor" type="ray">
                 <always_on>true</always_on>
                 <visualize>true</visualize>
-                <update_rate>20</update_rate>
+                <update_rate>100</update_rate>
                 <ray>
                     <radiation_type>infrared</radiation_type>
@@ -44,6 +44,6 @@
                             <samples>360</samples>
                             <resolution>1.000000</resolution>
-                            <min_angle>-0.523598776</min_angle>
-                            <max_angle>0.523598776</max_angle>
+                            <min_angle>-0.45</min_angle>
+                            <max_angle>0.45</max_angle>
                         </horizontal>
                     </scan>
@@ -62,4 +62,6 @@
                     <frame_name>left_tri_ir_range_frame</frame_name>
                     <radiation_type>infrared</radiation_type>
+                    <gaussianNoise>0.01</gaussianNoise>
+                    <updateRate>30</updateRate>
                 </plugin>
             </sensor>

File: src/swarm_process_robot/process_robot_description/urdf/sensors/tri_ir_sensor/tri_ir_sensor_middle.urdf.xacro (robot description, xacro)
@@ -29,13 +29,14 @@
         <joint name="tri_ir_range_joint" type="fixed">
             <axis xyz="0 0 0" />
-            <origin rpy="0 0 0" xyz="${0.01/2} 0 0" />
+            <origin rpy="0 0 0" xyz="${0.01/2+0.001} 0 0" />
             <parent link="tri_ir_sensor" />
             <child link="tri_ir_range_frame" />
         </joint>
-        <gazebo reference="tri_ir_sensor">
+        <!-- Specs https://www.pololu.com/product/3412 -->
+        <gazebo reference="tri_ir_range_frame">
             <sensor name="ir_sensor" type="ray">
                 <always_on>true</always_on>
                 <visualize>true</visualize>
-                <update_rate>20</update_rate>
+                <update_rate>100</update_rate>
                 <ray>
                     <radiation_type>infrared</radiation_type>
@@ -62,4 +63,6 @@
                     <frame_name>tri_ir_range_frame</frame_name>
                     <radiation_type>infrared</radiation_type>
+                    <gaussianNoise>0.01</gaussianNoise>
+                    <updateRate>30</updateRate>
                 </plugin>
             </sensor>

File: src/swarm_process_robot/process_robot_description/urdf/sensors/tri_ir_sensor/tri_ir_sensor_right.urdf.xacro (robot description, xacro)
@@ -29,13 +29,13 @@
         <joint name="right_tri_ir_range_joint" type="fixed">
             <axis xyz="0 0 0" />
-            <origin rpy="0 0 0" xyz="${0.01/2} 0 0" />
+            <origin rpy="0 0 0" xyz="${0.01/2+0.001} 0 0" />
             <parent link="right_tri_ir_sensor" />
             <child link="right_tri_ir_range_frame" />
         </joint>
-        <gazebo reference="right_tri_ir_sensor">
+        <gazebo reference="right_tri_ir_range_frame">
             <sensor name="right_ir_sensor" type="ray">
                 <always_on>true</always_on>
                 <visualize>true</visualize>
-                <update_rate>20</update_rate>
+                <update_rate>100</update_rate>
                 <ray>
                     <scan>
@@ -43,6 +43,6 @@
                             <samples>360</samples>
                             <resolution>1.000000</resolution>
-                            <min_angle>-0.523598776</min_angle>
-                            <max_angle>0.523598776</max_angle>
+                            <min_angle>-0.45</min_angle>
+                            <max_angle>0.45</max_angle>
                         </horizontal>
                     </scan>
@@ -61,4 +61,6 @@
                     <frame_name>right_tri_ir_range_frame</frame_name>
                     <radiation_type>infrared</radiation_type>
+                    <gaussianNoise>0.01</gaussianNoise>
+                    <updateRate>30</updateRate>
                 </plugin>
             </sensor>

Commit message: working navigation with real robot

File: src/swarm_process_robot/process_robot_description/urdf/process_robot.urdf.xacro (robot description, xacro)
@@ -13,6 +13,4 @@
   <xacro:include filename="$(find linorobot2_description)/urdf/mech/base.urdf.xacro" />
   <xacro:include filename="$(find linorobot2_description)/urdf/mech/mecanum_wheel.urdf.xacro" />
-  <xacro:include filename="$(find linorobot2_description)/urdf/sensors/generic_laser.urdf.xacro" />
-  <xacro:include filename="$(find linorobot2_description)/urdf/sensors/depth_sensor.urdf.xacro" />
   <!-- Assembly of robot -->
   <xacro:base
@@ -61,7 +59,7 @@
     />
   <xacro:imu/>
-  <xacro:tri_ir_sensor x="${base_length/2-0.20000}" y="0" z="${base_height/2+0.010}" roll="0" pitch="0" yaw="0" />
-  <xacro:left_tri_ir_sensor x="${base_length/2-0.20000}" y="0.01" z="${base_height/2+0.010}" roll="0" pitch="0" yaw="0" />
-  <xacro:right_tri_ir_sensor x="${base_length/2-0.20000}" y="-0.01" z="${base_height/2+0.010}" roll="0" pitch="0" yaw="0" />
+  <xacro:tri_ir_sensor x="${base_length/2}" y="0" z="${-base_height/2+0.010}" roll="0" pitch="0" yaw="0" />
+  <xacro:left_tri_ir_sensor x="${base_length/2}" y="0.01" z="${-base_height/2+0.010}" roll="0" pitch="0" yaw="0" />
+  <xacro:right_tri_ir_sensor x="${base_length/2}" y="-0.01" z="${-base_height/2+0.010}" roll="0" pitch="0" yaw="0" />
   <xacro:web_cam x="${base_length/2}" y="0" z="${base_height/2}" roll="0" pitch="0" yaw="0" />
   <xacro:omni_drive_controller/>

File: src/swarm_process_robot/process_robot_description/urdf/process_robot_properties.urdf.xacro (robot description, xacro)
@@ -1,13 +1,13 @@
 <?xml version="1.0"?>
 <robot xmlns:xacro="http://ros.org/wiki/xacro">
-  <xacro:property name="base_length" value="0.445" />
-  <xacro:property name="base_width" value="0.200" />
-  <xacro:property name="base_height" value="0.129" />
-  <xacro:property name="base_mass" value="10" />
-  <xacro:property name="wheel_radius" value="0.1" />
-  <xacro:property name="wheel_width" value="0.05" />
-  <xacro:property name="wheel_pos_x" value="0.120" />
-  <xacro:property name="wheel_pos_y" value="0.1355" />
-  <xacro:property name="wheel_pos_z" value="-0.04788" />
+  <xacro:property name="base_length" value="0.300" />
+  <xacro:property name="base_width" value="0.300" />
+  <xacro:property name="base_height" value="0.140" />
+  <xacro:property name="base_mass" value="5.0" />
+  <xacro:property name="wheel_radius" value="0.05" />
+  <xacro:property name="wheel_width" value="0.08" />
+  <xacro:property name="wheel_pos_x" value="0.100" />
+  <xacro:property name="wheel_pos_y" value="0.200" />
+  <xacro:property name="wheel_pos_z" value="-0.04" />
   <xacro:property name="wheel_mass" value=".4" />
   <xacro:property name="wheel_torque" value="20" />
