Commit message: tha big robot is working

File: src/swarm_process_robot/process_robot_description/urdf/process_robot_properties.urdf.xacro (robot description, xacro)
@@ -1,4 +1,20 @@
 <?xml version="1.0"?>
 <robot xmlns:xacro="http://ros.org/wiki/xacro">
+  <!-- Alu process bot -->
+  <xacro:property name="base_length" value="0.540" />
+  <xacro:property name="base_width" value="0.340" />
+  <xacro:property name="base_height" value="0.120" />
+  <xacro:property name="base_mass" value="5.0" />
+  <xacro:property name="wheel_radius" value="0.05" />
+  <xacro:property name="wheel_width" value="0.08" />
+  <xacro:property name="wheel_pos_x" value="0.209" />
+  <xacro:property name="wheel_pos_y" value="0.226" />
+  <xacro:property name="wheel_pos_z" value="-0.078" />
+  <xacro:property name="wheel_mass" value=".4" />
+  <xacro:property name="wheel_torque" value="20" />
+  340
+  540
+  <!-- Wood plate prototype -->
+  <!--
   <xacro:property name="base_length" value="0.300" />
   <xacro:property name="base_width" value="0.300" />
@@ -12,3 +28,4 @@
   <xacro:property name="wheel_mass" value=".4" />
   <xacro:property name="wheel_torque" value="20" />
+  -->
 </robot>
